Commit message: Collision meshes simplification WIP

File: urdf/tracer/tracer.urdf (robot description, URDF)
Before this commit: robot tracer_v1, 12 links, 11 joints
Links:
- link base_link: geometry visual mesh filename=meshes/tracer_base_link_no_wheel.dae
- link fl_wheel_link: geometry collision cylinder length=0.04653 radius=0.036; visual mesh filename=meshes/castor.dae
- link fr_wheel_link: geometry collision cylinder length=0.04653 radius=0.036; visual mesh filename=meshes/castor.dae
- link left_wheel_link: geometry collision cylinder length=0.0787019 radius=0.0605; visual mesh filename=meshes/tracer_wheel.dae
- link right_wheel_link: geometry collision cylinder length=0.0787019 radius=0.0605; visual mesh filename=meshes/tracer_wheel.dae
- link rl_wheel_link: geometry collision cylinder length=0.04653 radius=0.036; visual mesh filename=meshes/castor.dae
- link rr_wheel_link: geometry collision cylinder length=0.04653 radius=0.036; visual mesh filename=meshes/castor.dae

Commit message: All wheels replaced with cylinders

File: urdf/tracer/tracer.urdf (robot description, URDF)
Before this commit: robot tracer_v1, 12 links, 11 joints
Links:
- link fl_wheel_link: geometry collision cylinder length=0.04653 radius=0.036; visual cylinder length=0.04653 radius=0.036
- link fr_wheel_link: geometry collision cylinder length=0.04653 radius=0.036; visual cylinder length=0.04653 radius=0.036
- link left_wheel_link: geometry collision cylinder length=0.0787019 radius=0.0605; visual cylinder length=0.0787019 radius=0.0605
- link right_wheel_link: geometry collision cylinder length=0.0787019 radius=0.0605; visual cylinder length=0.0787019 radius=0.0605
- link rl_wheel_link: geometry collision cylinder length=0.04653 radius=0.036; visual cylinder length=0.04653 radius=0.036
- link rr_wheel_link: geometry collision cylinder length=0.04653 radius=0.036; visual cylinder length=0.04653 radius=0.036

Commit message: Staged updated to the model and script; original backup added

File: urdf/tracer/tracer.urdf (robot description, URDF)
Before this commit: robot tracer_v1, 12 links, 11 joints
Joints:
- joint left_wheel: origin xyz=0 0.17 -0.082 rpy=3.14 0 0 -> xyz=0 0.17 -0.082 rpy=0 0 0
